Commit message: box size adjusted

File: HW1/arm_description/urdf/arm.urdf.xacro (robot description, xacro)
@@ -14,5 +14,5 @@
     <collision>
       <geometry>
-        <mesh filename="package://arm_description/meshes/base_link.stl" scale="0.001 0.001 0.001"/>
+        <box size="0.0904 0.0901 0.08"/>
       </geometry>
       <origin rpy="0 0 0" xyz="0 0 0"/>
@@ -38,5 +38,5 @@
     <collision>
       <geometry>
-          <mesh filename="package://arm_description/meshes/base_turn.stl" scale="0.001 0.001 0.001"/>
+          <box size="0.06 0.0782 0.007"/>
         </geometry>
       <origin rpy="0 0 0" xyz="0 0 0"/>
@@ -63,5 +63,5 @@
     <collision>
       <geometry>
-          <mesh filename="package://arm_description/meshes/base_turn_table_rot.stl" scale="0.001 0.001 0.001"/>
+          <box size="0.056 0.0556 0.027"/>
         </geometry>
       <origin rpy="0 0 0" xyz="0 0 0"/>
@@ -86,5 +86,5 @@
     <collision>
       <geometry>
-          <mesh filename="package://arm_description/meshes/dyn.stl" scale="0.01 0.01 0.01"/>
+          <box size="0.07 0.032 0.04"/>
         </geometry>
       <origin rpy="0 0 0" xyz="0 0 0"/>
@@ -119,5 +119,5 @@
     <collision>
       <geometry>
-          <mesh filename="package://arm_description/meshes/f4_n_f3.stl" scale="0.001 0.001 0.001"/>
+          <box size="0.048 0.0916 0.0286"/>
         </geometry>
       <origin rpy="0 0 0" xyz="0 0 0"/>
@@ -142,5 +142,5 @@
     <collision>
       <geometry>
-          <mesh filename="package://arm_description/meshes/dyn.stl" scale="0.01 0.01 0.01"/>
+          <box size="0.07 0.032 0.04"/>
         </geometry>
       <origin rpy="0 0 0" xyz="0 0 0"/>
@@ -175,5 +175,5 @@
     <collision>
       <geometry>
-          <mesh filename="package://arm_description/meshes/f4_n_f3.stl" scale="0.001 0.001 0.001"/>
+          <box size="0.048 0.0916 0.0286"/>
         </geometry>
       <origin rpy="0 0 0" xyz="0 0 0"/>
@@ -197,5 +197,5 @@
     <collision>
       <geometry>
-          <mesh filename="package://arm_description/meshes/dyn.stl" scale="0.01 0.01 0.01"/>
+          <box size="0.07 0.032 0.04"/>
         </geometry>
       <origin rpy="0 0 0" xyz="0 0 0"/>
@@ -230,5 +230,5 @@
     <collision>
       <geometry>
-        <mesh filename="package://arm_description/meshes/wrist.stl" scale="0.001 0.001 0.001"/>
+        <box size="0.0482 0.0547 0.043"/>
       </geometry>
       <origin rpy="0 0 0" xyz="0 0 0"/>
@@ -253,5 +253,5 @@
     <collision>
       <geometry>
-          <mesh filename="package://arm_description/meshes/dyn.stl" scale="0.01 0.01 0.01"/>
+          <box size="0.07 0.032 0.04"/>
         </geometry>
       <origin rpy="0 0 0" xyz="0 0 0"/>
@@ -286,5 +286,5 @@
     <collision>
       <geometry>
-          <mesh filename="package://arm_description/meshes/the_crawer_base.stl" scale="0.001 0.001 0.001"/>
+          <box size="0.1044 0.0578 0.005"/>
         </geometry>
       <origin rpy="0 0 0" xyz="0 0 0"/>
@@ -312,5 +312,5 @@
     <collision>
       <geometry>
-          <mesh filename="package://arm_description/meshes/the_crawer.stl" scale="0.001 0.001 0.001"/>
+          <box size="0.09 0.05 0.06"/>
         </geometry>
       <origin rpy="0 0 0" xyz="0 0 0"/>
@@ -338,5 +338,5 @@
     <collision>
       <geometry>
-          <mesh filename="package://arm_description/meshes/the_crawer.stl" scale="0.001 0.001 0.001"/>
+          <box size="0.09 0.05 0.06"/>
         </geometry>
       <origin rpy="0 0 0" xyz="0 0 0"/>

Commit message: aggiustata camera

File: HW1/arm_description/urdf/arm.urdf.xacro (robot description, xacro)
@@ -347,5 +347,5 @@
     </inertial>
   </link>
-  <xacro:include filename="$(find arm_description)/urdf/cam_tot.xacro"/>
+  <xacro:include filename="$(find arm_gazebo)/urdf/cam_tot.xacro"/>
   <xacro:my_camera parent="base_link"/>
   <gazebo>

File: HW1/arm_gazebo/urdf/cam_tot.xacro (robot description, xacro)
@@ -5,12 +5,14 @@
       <parent link="${parent}"/>
       <child link="camera_link"/>
-      <origin xyz="0.0 0 0.00" rpy="0.0 -1.57 0"/>
+      <origin xyz="0.001 -0.04 0.055" rpy="0.0 0.0 -1.57"/>
     </joint>
     <link name="camera_link">
       <visual>
         <geometry>
-          <box size="0.1 0.1 0.1"/>
+          <box size="0.01 0.01 0.01"/>
         </geometry>
-        <material name="red"/>
+          <material name="blue">
+            <color rgba="0 0 1 1"/>
+          </material>
       </visual>
     </link>

Commit message: box di nuovo

File: HW1/arm_description/urdf/arm.urdf.xacro (robot description, xacro)
@@ -14,5 +14,5 @@
     <collision>
       <geometry>
-        <mesh filename="package://arm_description/meshes/base_link.stl" scale="0.001 0.001 0.001"/>
+        <box size="0.0904 0.0901 0.08"/>
       </geometry>
       <origin rpy="0 0 0" xyz="0 0 0"/>
@@ -38,5 +38,5 @@
     <collision>
       <geometry>
-          <mesh filename="package://arm_description/meshes/base_turn.stl" scale="0.001 0.001 0.001"/>
+          <box size="0.06 0.0782 0.007"/>
         </geometry>
       <origin rpy="0 0 0" xyz="0 0 0"/>
@@ -63,5 +63,5 @@
     <collision>
       <geometry>
-          <mesh filename="package://arm_description/meshes/base_turn_table_rot.stl" scale="0.001 0.001 0.001"/>
+          <box size="0.056 0.0556 0.027"/>
         </geometry>
       <origin rpy="0 0 0" xyz="0 0 0"/>
@@ -86,5 +86,5 @@
     <collision>
       <geometry>
-          <mesh filename="package://arm_description/meshes/dyn.stl" scale="0.01 0.01 0.01"/>
+          <box size="0.07 0.032 0.04"/>
         </geometry>
       <origin rpy="0 0 0" xyz="0 0 0"/>
@@ -119,5 +119,5 @@
     <collision>
       <geometry>
-          <mesh filename="package://arm_description/meshes/f4_n_f3.stl" scale="0.001 0.001 0.001"/>
+          <box size="0.048 0.0916 0.0286"/>
         </geometry>
       <origin rpy="0 0 0" xyz="0 0 0"/>
@@ -142,5 +142,5 @@
     <collision>
       <geometry>
-          <mesh filename="package://arm_description/meshes/dyn.stl" scale="0.01 0.01 0.01"/>
+          <box size="0.07 0.032 0.04"/>
         </geometry>
       <origin rpy="0 0 0" xyz="0 0 0"/>
@@ -175,5 +175,5 @@
     <collision>
       <geometry>
-          <mesh filename="package://arm_description/meshes/f4_n_f3.stl" scale="0.001 0.001 0.001"/>
+          <box size="0.048 0.0916 0.0286"/>
         </geometry>
       <origin rpy="0 0 0" xyz="0 0 0"/>
@@ -197,5 +197,5 @@
     <collision>
       <geometry>
-          <mesh filename="package://arm_description/meshes/dyn.stl" scale="0.01 0.01 0.01"/>
+          <box size="0.07 0.032 0.04"/>
         </geometry>
       <origin rpy="0 0 0" xyz="0 0 0"/>
@@ -230,5 +230,5 @@
     <collision>
       <geometry>
-        <mesh filename="package://arm_description/meshes/wrist.stl" scale="0.001 0.001 0.001"/>
+        <box size="0.0482 0.0547 0.043"/>
       </geometry>
       <origin rpy="0 0 0" xyz="0 0 0"/>
@@ -253,5 +253,5 @@
     <collision>
       <geometry>
-          <mesh filename="package://arm_description/meshes/dyn.stl" scale="0.01 0.01 0.01"/>
+          <box size="0.07 0.032 0.04"/>
         </geometry>
       <origin rpy="0 0 0" xyz="0 0 0"/>
@@ -286,5 +286,5 @@
     <collision>
       <geometry>
-          <mesh filename="package://arm_description/meshes/the_crawer_base.stl" scale="0.001 0.001 0.001"/>
+          <box size="0.1044 0.0578 0.005"/>
         </geometry>
       <origin rpy="0 0 0" xyz="0 0 0"/>
@@ -312,5 +312,5 @@
     <collision>
       <geometry>
-          <mesh filename="package://arm_description/meshes/the_crawer.stl" scale="0.001 0.001 0.001"/>
+          <box size="0.09 0.05 0.06"/>
         </geometry>
       <origin rpy="0 0 0" xyz="0 0 0"/>
@@ -338,5 +338,5 @@
     <collision>
       <geometry>
-          <mesh filename="package://arm_description/meshes/the_crawer.stl" scale="0.001 0.001 0.001"/>
+          <box size="0.09 0.05 0.06"/>
         </geometry>
       <origin rpy="0 0 0" xyz="0 0 0"/>

File: HW1/arm_gazebo/urdf/cam_tot.xacro (robot description, xacro)
@@ -5,9 +5,5 @@
       <parent link="${parent}"/>
       <child link="camera_link"/>
-<<<<<<< HEAD:HW1/arm_gazebo/urdf/cam_tot.xacro
       <origin xyz="0.001 -0.04 0.055" rpy="0.0 0.0 -1.57"/>
-=======
-      <origin xyz="0.001 -0.04 0.055" rpy="0.0 -1.57 0"/>
->>>>>>> a71709e1f2620dd58e02cc182511721360c69a44:HW1/arm_description/urdf/cam_tot.xacro
     </joint>
     <link name="camera_link">
